File: main_board/main_board.kicad_sch (KiCad schematic)
At the start: 56 parts, among them J1 USB4105-GF-A-060, J2 Conn_01x06_Pin, Q3 NX3008PBK,215, U1 SSD1306, U2 ESP32-S2-SOLO, U3 TLV62568PDRLT, U4 MCP73832, U5 DW01, U6 8205A, U7 MAX17055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

Commit message: Tweak routing
Parts:
- R12: value 470k -> 5k1
- R13: value 1M -> 10k
Connections:
- net GND: now also U2.16 (IO46), U2.17 (IO9), U2.18 (IO10), U2.19 (IO11), U2.20 (IO12), U2.21 (IO13), U2.22 (IO14), U2.23 (IO21), U2.24 (IO33), U2.25 (IO34)
- no-connect marks 17 -> 7
Other:
- note added: "CHG_STAT: add internal pullup"
- note added: "ESP32-C6-WROOM No bottom pin row Strapping pins: - IO17: initially high - IO0: high for normal boot - IO42: ignored (high to use USB-JTAG) SPI: 1 + PARL_IO"
- note added: "ESP32-S2-SOLO Do not use bottom pin row Strapping pins: - IO0: high for normal boot - IO46: low - IO45: low SPI: 2"
- note added: "ESP32-S3-WROOM Do not use bottom pin row Strapping pins: - IO0: high for normal boot - IO45/IO46: low - IO3: ignored (high to use USB-JTAG) SPI: 2"
- note added: "Pins in these notes are written according to their position relative to the S2 module in the schematic. The actual pin names differ on different modules."
- note added: "S2: IO33, IO34 S3: IO47, IO48"
- note removed: "CHG_STAT: internal pullup"
- note removed: "S2: IO33, IO34 S3: IO46, IO47"
Changed lines of the file:
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@@
   (junction (at 110.49 55.88) (diameter 0) (color 0 0 0 0)
   )
+  (junction (at 158.75 78.74) (diameter 0) (color 0 0 0 0)
+  )
   (junction (at 113.03 139.7) (diameter 0) (color 0 0 0 0)
   )
@@
   (junction (at 129.54 186.69) (diameter 0) (color 0 0 0 0)
   )
+  (junction (at 151.13 78.74) (diameter 0) (color 0 0 0 0)
+  )
   (junction (at 240.03 147.32) (diameter 0) (color 0 0 0 0)
   )
@@
   (junction (at 248.92 128.27) (diameter 0) (color 0 0 0 0)
   )
+  (junction (at 143.51 78.74) (diameter 0) (color 0 0 0 0)
+  )
+  (junction (at 163.83 78.74) (diameter 0) (color 0 0 0 0)
+  )
   (junction (at 102.87 71.12) (diameter 0) (color 0 0 0 0)
   )
@@
   (junction (at 121.92 186.69) (diameter 0) (color 0 0 0 0)
   )
+  (junction (at 146.05 78.74) (diameter 0) (color 0 0 0 0)
+  )
   (junction (at 246.38 78.74) (diameter 0) (color 0 0 0 0)
   )
@@
   (junction (at 212.09 143.51) (diameter 0) (color 0 0 0 0)
   )
+  (junction (at 140.97 78.74) (diameter 0) (color 0 0 0 0)
+  )
   (junction (at 97.79 35.56) (diameter 0) (color 0 0 0 0)
   )
@@
   (junction (at 78.74 148.59) (diameter 0) (color 0 0 0 0)
   )
+  (junction (at 161.29 78.74) (diameter 0) (color 0 0 0 0)
+  )
   (junction (at 248.92 113.03) (diameter 0) (color 0 0 0 0)
   )
+  (junction (at 153.67 78.74) (diameter 0) (color 0 0 0 0)
+  )
   (junction (at 246.38 147.32) (diameter 0) (color 0 0 0 0)
   )
@@
   (junction (at 115.57 148.59) (diameter 0) (color 0 0 0 0)
   )
+  (junction (at 156.21 78.74) (diameter 0) (color 0 0 0 0)
+  )
   (junction (at 64.77 165.1) (diameter 0) (color 0 0 0 0)
   )
@@
   (junction (at 38.1 151.13) (diameter 0) (color 0 0 0 0)
   )
+  (junction (at 138.43 78.74) (diameter 0) (color 0 0 0 0)
+  )
   (junction (at 248.92 120.65) (diameter 0) (color 0 0 0 0)
   )
@@
   (junction (at 248.92 124.46) (diameter 0) (color 0 0 0 0)
   )
+  (junction (at 148.59 78.74) (diameter 0) (color 0 0 0 0)
+  )
   (junction (at 74.93 121.92) (diameter 0) (color 0 0 0 0)
   )
@@
   (junction (at 102.87 55.88) (diameter 0) (color 0 0 0 0)
   )
-  (no_connect (at 158.75 78.74))
   (no_connect (at 254 109.22))
-  (no_connect (at 138.43 78.74))
-  (no_connect (at 153.67 78.74))
   (no_connect (at 198.12 144.78))
-  (no_connect (at 148.59 78.74))
   (no_connect (at 139.7 170.18))
-  (no_connect (at 143.51 78.74))
-  (no_connect (at 161.29 78.74))
   (no_connect (at 139.7 172.72))
-  (no_connect (at 146.05 78.74))
-  (no_connect (at 140.97 78.74))
   (no_connect (at 198.12 147.32))
   (no_connect (at 81.28 162.56))
   (no_connect (at 170.18 50.8))
-  (no_connect (at 151.13 78.74))
-  (no_connect (at 156.21 78.74))
   (wire (pts (xy 116.84 58.42) (xy 129.54 58.42))
     (stroke (width 0) (type default))
@@
     (stroke (width 0) (type default))
   )
+  (wire (pts (xy 156.21 78.74) (xy 158.75 78.74))
+    (stroke (width 0) (type default))
+  )
   (wire (pts (xy 170.18 38.1) (xy 179.07 38.1))
     (stroke (width 0) (type default))
@@
     (stroke (width 0) (type default))
   )
+  (wire (pts (xy 146.05 78.74) (xy 148.59 78.74))
+    (stroke (width 0) (type default))
+  )
   (wire (pts (xy 200.66 45.72) (xy 200.66 55.88))
     (stroke (width 0) (type default))
@@
     (stroke (width 0) (type default))
   )
+  (wire (pts (xy 138.43 78.74) (xy 138.43 80.01))
+    (stroke (width 0) (type default))
+  )
   (wire (pts (xy 240.03 147.32) (xy 246.38 147.32))
     (stroke (width 0) (type default))
@@
     (stroke (width 0) (type default))
   )
+  (wire (pts (xy 148.59 78.74) (xy 151.13 78.74))
+    (stroke (width 0) (type default))
+  )
   (wire (pts (xy 204.47 110.49) (xy 215.9 110.49))
     (stroke (width 0) (type default))
@@
     (stroke (width 0) (type default))
   )
+  (wire (pts (xy 143.51 78.74) (xy 146.05 78.74))
+    (stroke (width 0) (type default))
+  )
   (wire (pts (xy 26.67 151.13) (xy 26.67 165.1))
     (stroke (width 0) (type default))
@@
     (stroke (width 0) (type default))
   )
+  (wire (pts (xy 140.97 78.74) (xy 143.51 78.74))
+    (stroke (width 0) (type default))
+  )
   (wire (pts (xy 69.85 53.34) (xy 85.09 53.34))
     (stroke (width 0) (type default))
@@
     (stroke (width 0) (type default))
   )
+  (wire (pts (xy 153.67 78.74) (xy 156.21 78.74))
+    (stroke (width 0) (type default))
+  )
   (wire (pts (xy 200.66 135.89) (xy 200.66 137.16))
     (stroke (width 0) (type default))
@@
     (stroke (width 0) (type default))
   )
+  (wire (pts (xy 158.75 78.74) (xy 161.29 78.74))
+    (stroke (width 0) (type default))
+  )
   (wire (pts (xy 25.4 194.31) (xy 43.18 194.31))
     (stroke (width 0) (type default))
@@
     (stroke (width 0) (type default))
   )
+  (wire (pts (xy 151.13 78.74) (xy 153.67 78.74))
+    (stroke (width 0) (type default))
+  )
   (wire (pts (xy 246.38 139.7) (xy 254 139.7))
     (stroke (width 0) (type default))
@@
     (stroke (width 0) (type default))
   )
+  (wire (pts (xy 138.43 78.74) (xy 140.97 78.74))
+    (stroke (width 0) (type default))
+  )
   (wire (pts (xy 246.38 71.12) (xy 246.38 74.93))
     (stroke (width 0) (type default))
@@
     (stroke (width 0) (type default))
   )
+  (wire (pts (xy 161.29 78.74) (xy 163.83 78.74))
+    (stroke (width 0) (type default))
+  )
   (wire (pts (xy 195.58 45.72) (xy 195.58 48.26))
     (stroke (width 0) (type default))
@@
     (effects (font (size 1.27 1.27)) (justify left bottom))
   )
+  (text "ESP32-C6-WROOM\nNo bottom pin row\nStrapping pins:\n - IO17: initially high\n - IO0: high for normal boot\n - IO42: ignored (high to use USB-JTAG)\nSPI: 1 + PARL_IO"
+    (at 161.29 -25.4 0)
+    (effects (font (size 1.27 1.27)) (justify left bottom))
+  )
   (text "Kelvin-connect CSP and CSN to R18" (at 128.27 194.945 0)
     (effects (font (size 1.27 1.27)) (justify left bottom))
   )
+  (text "ESP32-S3-WROOM\nDo not use bottom pin row\nStrapping pins:\n - IO0: high for normal boot\n - IO45/IO46: low\n - IO3: ignored (high to use USB-JTAG)\nSPI: 2"
+    (at 114.3 -25.4 0)
+    (effects (font (size 1.27 1.27)) (justify left bottom))
+  )
   (text "Battery charger" (at 14.605 140.335 0)
     (effects (font (size 1.27 1.27)) (justify left bottom))
   )
-  (text "CHG_STAT: internal pullup" (at 148.59 100.965 0)
+  (text "ESP32-S2-SOLO\nDo not use bottom pin row\nStrapping pins:\n - IO0: high for normal boot\n - IO46: low\n - IO45: low\nSPI: 2"
+    (at 77.47 -25.4 0)
+    (effects (font (size 1.27 1.27)) (justify left bottom))
+  )
+  (text "CHG_STAT: add \ninternal pullup" (at 196.85 67.31 0)
+    (effects (font (size 1.27 1.27)) (justify left bottom))
+  )
+  (text "Pins in these notes are written according\nto their position relative to the S2 module\nin the schematic. The actual pin names\ndiffer on different modules."
+    (at 115.57 -50.8 0)
     (effects (font (size 1.27 1.27)) (justify left bottom))
   )
@@
     (effects (font (size 1.27 1.27)) (justify left bottom))
   )
-  (text "45-46: strapping pins, don't use" (at 148.59 98.425 0)
+  (text "45-46: strapping pins, don't use" (at 142.24 88.9 0)
     (effects (font (size 1.27 1.27)) (justify left bottom))
   )
@@
     (effects (font (size 1.27 1.27)) (justify left bottom))
   )
-  (text "S2: IO33, IO34\nS3: IO46, IO47" (at 167.005 76.2 0)
+  (text "S2: IO33, IO34\nS3: IO47, IO48" (at 167.005 76.2 0)
     (effects (font (size 1.27 1.27)) (justify left bottom))
   )
   (text "IO3 ignored unless\nEFUSE_STRAP_JTAG_SEL = 1\nGND=JTAG\n3V3=USB"
-    (at 111.76 87.63 0)
+    (at 109.22 86.36 0)
     (effects (font (size 1.27 1.27)) (justify left bottom))
   )
@@
     )
   )
+  (symbol (lib_id "power:GND") (at 138.43 80.01 0) (unit 1)
+    (in_bom yes) (on_board yes) (dnp no) (fields_autoplaced)
+    (property "Reference" "#PWR040" (at 138.43 86.36 0)
+      (effects (font (size 1.27 1.27)) hide)
+    )
+    (property "Value" "GND" (at 138.43 85.09 0)
+      (effects (font (size 1.27 1.27)))
+    )
+    (property "Footprint" "" (at 138.43 80.01 0)
+      (effects (font (size 1.27 1.27)) hide)
+    )
+    (property "Datasheet" "" (at 138.43 80.01 0)
+      (effects (font (size 1.27 1.27)) hide)
+    )
+    (pin "1")
+    (instances
+      (project "main_board"
+        (path "/e55848cd-275a-4b5e-8e68-b5d8d07c8d31"
+          (reference "#PWR040") (unit 1)
+        )
+      )
+    )
+  )
   (symbol (lib_id "Device:R") (at 69.85 165.1 90) (mirror x) (unit 1)
     (in_bom yes) (on_board yes) (dnp no)
@@
       (effects (font (size 1.27 1.27)) (justify left))
     )
-    (property "Value" "1M" (at 214.63 149.225 0)
+    (property "Value" "10k" (at 214.63 149.225 0)
       (effects (font (size 1.27 1.27)) (justify left))
     )
@@
       (effects (font (size 1.27 1.27)) (justify left))
     )
-    (property "Value" "470k" (at 213.995 139.7 0)
+    (property "Value" "5k1" (at 213.995 139.7 0)
       (effects (font (size 1.27 1.27)) (justify left))
     )
